Commit message: feat: support wuji fix bug

File: OmniGibson/omnigibson/adept/custom_assets/r1pro_wuji/urdf/r1pro_wuji.urdf (robot description, URDF)
Before this commit: robot r1pro_wuji, 104 links, 103 joints
Links:
- removed link l_index_finger_tip
- removed link l_middle_finger_tip
- removed link l_pinky_tip
- removed link l_ring_finger_tip
- removed link l_thumb_tip
- removed link r_index_finger_tip
- removed link r_middle_finger_tip
- removed link r_pinky_tip
- removed link r_ring_finger_tip
- removed link r_thumb_tip
- link left_realsense_link: geometry visual box size=0.001 0.001 0.001
- link right_realsense_link: geometry visual box size=0.001 0.001 0.001
- link zed_link: geometry visual box size=0.001 0.001 0.001
Joints:
- removed joint l_index_finger_tip_fixed
- removed joint l_middle_finger_tip_fixed
- removed joint l_pinky_tip_fixed
- removed joint l_ring_finger_tip_fixed
- removed joint l_thumb_tip_fixed
- removed joint r_index_finger_tip_fixed
- removed joint r_middle_finger_tip_fixed
- removed joint r_pinky_tip_fixed
- removed joint r_ring_finger_tip_fixed
- removed joint r_thumb_tip_fixed
- joint camera_head_left_joint: axis 0 0 0 -> (none)
- joint camera_head_right_joint: axis 0 0 0 -> (none)
- joint head_joint: axis 0 0 0 -> (none)
- joint imu_chassis_joint: axis 0 0 0 -> (none)
- joint imu_torso_joint: axis 0 0 0 -> (none)
- joint left_arm_base_joint: axis 0 0 0 -> (none)
- joint left_d405_joint: axis 0 0 0 -> (none)
- joint left_gmsl_joint: axis 0 0 0 -> (none)
- joint lidar_chassis_left_joint: axis 0 0 0 -> (none)
- joint right_arm_base_joint: axis 0 0 0 -> (none)
- joint right_d405_joint: axis 0 0 0 -> (none)
- joint right_gmsl_joint: axis 0 0 0 -> (none)

Commit message: feat: support wuji fix bug

File: OmniGibson/omnigibson/adept/custom_assets/r1pro_wuji/urdf/r1pro_wuji.urdf (robot description, URDF)
Before this commit: robot r1pro_wuji, 94 links, 93 joints
Joints:
- joint l_mount_joint: origin xyz=-0.0295 0 -0.1637 rpy=0 0 0 -> xyz=-0.0295 0 -0.1637 rpy=0 0 1.570796327
- joint left_d405_joint: origin xyz=0.045176 0.009 -0.141517 rpy=2.4435 0 -1.5708 -> xyz=0.074676 0.009 0.022183 rpy=2.4435 0 -1.5708; parent left_arm_link7 -> l_mount
- joint left_gmsl_joint: origin xyz=0.03179 0 -0.1554115 rpy=-3.1416 0 -1.5708 -> xyz=0.06129 0 0.0082885 rpy=-3.1416 0 -1.5708; parent left_arm_link7 -> l_mount
- joint left_realsense_joint: origin xyz=0.045176 0.009 -0.141517 rpy=2.4435 0 -1.5708 -> xyz=0.074676 0.009 0.022183 rpy=2.4435 0 -1.5708; parent left_arm_link7 -> l_mount
- joint r_mount_joint: origin xyz=-0.0295 0 -0.1637 rpy=0 0 0 -> xyz=-0.0295 0 -0.1637 rpy=0 0 1.570796327
- joint right_d405_joint: origin xyz=0.045176 0.009 -0.141517 rpy=2.4435 0 -1.5708 -> xyz=0.074676 0.009 0.022183 rpy=2.4435 0 -1.5708; parent right_arm_link7 -> r_mount
- joint right_gmsl_joint: origin xyz=0.03179 0 -0.1554115 rpy=-3.1416 0 -1.5708 -> xyz=0.06129 0 0.0082885 rpy=-3.1416 0 -1.5708; parent right_arm_link7 -> r_mount
- joint right_realsense_joint: origin xyz=0.045176 0.009 -0.141517 rpy=2.4435 0 -1.5708 -> xyz=0.074676 0.009 0.022183 rpy=2.4435 0 -1.5708; parent right_arm_link7 -> r_mount
- joint zed_joint: origin xyz=0.064821 -0.0001785 0.093658 rpy=0 0 0 -> xyz=0.064821 -0.0001785 0.093658 rpy=-1.9199 0 -1.5708

Commit message: feat: support wuji fix bug

File: OmniGibson/omnigibson/adept/custom_assets/r1pro_wuji/urdf/r1pro_wuji.urdf (robot description, URDF)
Before this commit: robot r1pro_wuji, 94 links, 93 joints
Links:
- added link left_gripper_link, mass 0.0934809943288547; visual mesh filename=../meshes/r1pro/left_gripper_link.STL
- added link right_gripper_link, mass 0.24625; visual mesh filename=../meshes/r1pro/left_gripper_link.STL
Joints:
- added joint left_gripper_joint: type fixed, parent left_arm_link7, child left_gripper_link, origin xyz=-0.0295 0.0 -0.1637 rpy=0 0 0
- added joint right_gripper_joint: type fixed, parent right_arm_link7, child right_gripper_link, origin xyz=-0.0295 0.0 -0.1637 rpy=0 0 0

Commit message: feat: support wuji fix bug

File: OmniGibson/omnigibson/adept/custom_assets/r1pro_wuji/urdf/r1pro_wuji.urdf (robot description, URDF)
Before this commit: robot r1pro_wuji, 96 links, 95 joints
Links:
- removed link left_d405_link
- removed link left_gmsl_link
- removed link right_d405_link
- removed link right_gmsl_link
- link base_link: geometry collision mesh filename=../meshes/r1pro/base_link.STL; visual mesh filename=../meshes/textured/base_link.obj
- link left_arm_base_link: geometry collision mesh filename=../meshes/r1pro/left_arm_base_link.STL; visual mesh filename=../meshes/textured/left_arm_base_link.obj
- link left_arm_link1: geometry collision mesh filename=../meshes/r1pro/left_arm_link1.STL; visual mesh filename=../meshes/textured/left_arm_link1.obj
- link left_arm_link2: geometry collision mesh filename=../meshes/r1pro/left_arm_link2.STL; visual mesh filename=../meshes/textured/left_arm_link2.obj
- link left_arm_link3: geometry collision mesh filename=../meshes/r1pro/left_arm_link3.STL; visual mesh filename=../meshes/textured/left_arm_link3.obj
- link left_arm_link4: geometry collision mesh filename=../meshes/r1pro/left_arm_link4.STL; visual mesh filename=../meshes/textured/left_arm_link4.obj
- link left_arm_link5: geometry collision mesh filename=../meshes/r1pro/left_arm_link5.STL; visual mesh filename=../meshes/textured/left_arm_link5.obj
- link left_arm_link6: geometry collision mesh filename=../meshes/r1pro/left_arm_link6.STL; visual mesh filename=../meshes/textured/left_arm_link6.obj
- link left_arm_link7: geometry collision mesh filename=../meshes/r1pro/left_arm_link7.STL; visual mesh filename=../meshes/textured/left_arm_link7.obj
- link left_gripper_link: geometry visual mesh filename=../meshes/textured/left_gripper_link.obj
- link left_realsense_link: geometry visual mesh filename=../meshes/textured/left_realsense_link.obj
- link right_arm_base_link: geometry collision mesh filename=../meshes/r1pro/right_arm_base_link.STL; visual mesh filename=../meshes/textured/right_arm_base_link.obj
- link right_arm_link1: geometry collision mesh filename=../meshes/r1pro/right_arm_link1.STL; visual mesh filename=../meshes/textured/right_arm_link1.obj
- link right_arm_link2: geometry collision mesh filename=../meshes/r1pro/right_arm_link2.STL; visual mesh filename=../meshes/textured/right_arm_link2.obj
- link right_arm_link3: geometry collision mesh filename=../meshes/r1pro/right_arm_link3.STL; visual mesh filename=../meshes/textured/right_arm_link3.obj
- link right_arm_link4: geometry collision mesh filename=../meshes/r1pro/right_arm_link4.STL; visual mesh filename=../meshes/textured/right_arm_link4.obj
- link right_arm_link5: geometry collision mesh filename=../meshes/r1pro/right_arm_link5.STL; visual mesh filename=../meshes/textured/right_arm_link5.obj
- link right_arm_link6: geometry collision mesh filename=../meshes/r1pro/right_arm_link6.STL; visual mesh filename=../meshes/textured/right_arm_link6.obj
- link right_arm_link7: geometry collision mesh filename=../meshes/r1pro/right_arm_link7.STL; visual mesh filename=../meshes/textured/right_arm_link7.obj
- link right_gripper_link: geometry visual mesh filename=../meshes/textured/right_gripper_link.obj
- link right_realsense_link: geometry visual mesh filename=../meshes/textured/right_realsense_link.obj
- link steer_motor_link1: geometry collision mesh filename=../meshes/r1pro/steer_motor_link1.STL; visual mesh filename=../meshes/textured/steer_motor_link1.obj
- link steer_motor_link2: geometry collision mesh filename=../meshes/r1pro/steer_motor_link2.STL; visual mesh filename=../meshes/textured/steer_motor_link2.obj
- link steer_motor_link3: geometry collision mesh filename=../meshes/r1pro/steer_motor_link3.STL; visual mesh filename=../meshes/textured/steer_motor_link3.obj
- link torso_link1: geometry collision mesh filename=../meshes/r1pro/torso_link1.STL; visual mesh filename=../meshes/textured/torso_link1.obj
- link torso_link2: geometry collision mesh filename=../meshes/r1pro/torso_link2.STL; visual mesh filename=../meshes/textured/torso_link2.obj
- link torso_link3: geometry collision mesh filename=../meshes/r1pro/torso_link3.STL; visual mesh filename=../meshes/textured/torso_link3.obj
- link torso_link4: geometry collision mesh filename=../meshes/r1pro/torso_link4.STL; visual mesh filename=../meshes/textured/torso_link4.obj
- link wheel_motor_link1: geometry collision mesh filename=../meshes/r1pro/wheel_motor_link1.STL; visual mesh filename=../meshes/textured/wheel_motor_link1.obj
- link wheel_motor_link2: geometry collision mesh filename=../meshes/r1pro/wheel_motor_link2.STL; visual mesh filename=../meshes/textured/wheel_motor_link2.obj
- link wheel_motor_link3: geometry collision mesh filename=../meshes/r1pro/wheel_motor_link3.STL; visual mesh filename=../meshes/textured/wheel_motor_link3.obj
- link zed_link: geometry visual mesh filename=../meshes/textured/zed_link.obj
Joints:
- removed joint left_d405_joint
- removed joint left_gmsl_joint
- removed joint right_d405_joint
- removed joint right_gmsl_joint
- joint l_mount_joint: origin xyz=-0.0295 0 -0.1637 rpy=0 0 1.570796327 -> xyz=-0.0295 0 -0.1637 rpy=0 0 -1.570796327
- joint left_realsense_joint: origin xyz=0.074676 0.009 0.022183 rpy=2.4435 0 -1.5708 -> xyz=0.05051 0.0028934 0.0051317 rpy=-3.1376 -0.43631 3.1399; parent l_mount -> left_gripper_link
- joint right_realsense_joint: origin xyz=0.074676 0.009 0.022183 rpy=2.4435 0 -1.5708 -> xyz=0.05051 0.0028934 0.0051317 rpy=-3.1376 -0.43631 3.1399; parent r_mount -> right_gripper_link
- joint zed_joint: origin xyz=0.064821 -0.0001785 0.093658 rpy=-1.9199 0 -1.5708 -> xyz=0.065511 0.060003 0.47598 rpy=-1.9199 0 -1.5708; parent head_link -> torso_link4
